File: Matias.kicad_sch (KiCad schematic)
At the start: 0 parts

Commit message: Finish schematics and layout
Parts:
- added C1, C5: 100n, Capacitor_SMD:C_0603_1608Metric, symbol Device:C
- added C10, C9: 10u, Capacitor_SMD:C_0603_1608Metric, symbol Device:C
- added C2, C3, C4: 10u, Capacitor_SMD:C_0805_2012Metric, symbol Device:C
- added C6, C7: 47u, Capacitor_THT:CP_Radial_D5.0mm_P2.00mm, symbol Device:C_Polarized
- added C8: 270u, Capacitor_THT:CP_Radial_D6.3mm_P2.50mm, symbol Device:C_Polarized
- added D1, D2, D3: LED, LED_SMD:LED_0603_1608Metric, symbol Device:LED
- added IC1: TPS65133DPDR, Components:SON45P300X300X80-13N-D, symbol TPS65133DPDR:TPS65133DPDR
- added IC3: OPA1677DBVR, Components:SOT95P280X145-5N, symbol OPA1677DBVR:OPA1677DBVR
- added J1: Conn_01x03_Pin, Connector_PinHeader_2.54mm:PinHeader_1x03_P2.54mm_Vertical, symbol Connector:Conn_01x03_Pin
- added J2, J3: Conn_01x02_Pin, Connector_PinHeader_2.54mm:PinHeader_1x02_P2.54mm_Vertical, symbol Connector:Conn_01x02_Pin
- added L1, L2: 4.7uH, Inductor_SMD:L_1008_2520Metric, symbol Device:L
- added R1: 100k, Resistor_SMD:R_0603_1608Metric, symbol Device:R
- added R2, R3: 10k, Resistor_SMD:R_0603_1608Metric, symbol Device:R
- added R4, R6, R7: 300, Resistor_SMD:R_0603_1608Metric, symbol Device:R
- added VR1: PVG3A104C01R00, PVG3A104C01R00, symbol PVG3A104C01R00:PVG3A104C01R00
Connections:
- new net: IC3.4 (-IN), R2.1, R3.1, VR1.2 (WI[ER)
- new net: C7.2, R3.2
- new net: D2.2 (A), R6.1
- new net: C6.1, J1.3 (Pin_3)
- new net: C6.2, R2.2
- new net: C8.2, J3.1 (Pin_1)
- new net: C5.1, IC1.7 (EN), R1.2
- new net: C7.1, J1.1 (Pin_1)
- new net: D3.1 (K), R7.1
- new net: C8.1, IC3.1 (OUT), VR1.1 (CCW)
- new net: IC1.1 (SWP), L2.1
- new net: D1.1 (K), R4.1
- new net +5V: C1.1, C4.1, D1.2 (A), IC1.11 (AVIN), IC1.12 (PVIN), J2.2 (Pin_2), L2.2, R1.1
- new net GND: C1.2, C10.2, C2.2, C3.2, C4.2, C5.2, C9.2, IC1.13 (GND_4), IC1.2 (PGND), IC1.4 (GND_1), IC1.5 (AGND), IC1.6 (GND_2), IC1.8 (GND_3), IC3.3 (+IN), J1.2 (Pin_2), J2.1 (Pin_1), J3.2 (Pin_2), L1.2, R4.2, R6.2, R7.2
- new net SWN: IC1.10 (SWN), L1.1
- new net V+: C10.1, C3.1, D3.2 (A), IC1.3 (VPOS), IC3.5 (V+)
- new net V-: C2.1, C9.1, D2.1 (K), IC1.9 (VNEG), IC3.2 (V-)
- no-connect marks 0 -> 1
